File: Boopsie v1 Kicad Files/Boopsie v1.kicad_pcb (KiCad board)
At the start: 2 copper layers, 81 x 94.1 mm, 34 parts, among them J1 OLED_128x64, SW1 RotaryEncoder_Switch, SW2 RotaryEncoder_Switch, U1 RP2040_Zero

Commit message: pcb update
Routing:
- net Net-(D10-K): track 127.1 -> 125.0 mm
Changed lines of the file:
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@@
 			(outputformat 1)
 			(mirror no)
-			(drillshape 1)
+			(drillshape 0)
 			(scaleselection 1)
-			(outputdirectory "")
+			(outputdirectory "../Boopsie/Boopsie v1 Gerbers/")
 		)
 	)
@@
 			(at 0 -3.2 0)
 			(layer "F.SilkS")
+			(hide yes)
 			(effects
 				(font
@@
 			(at 0 3.2 0)
 			(layer "F.Fab")
+			(hide yes)
 			(effects
 				(font
@@
 			(at 0 -3.2 0)
 			(layer "F.SilkS")
+			(hide yes)
 			(effects
 				(font
@@
 			(at 0 3.2 0)
 			(layer "F.Fab")
+			(hide yes)
 			(effects
 				(font
@@
 			(at 0 -3.2 0)
 			(layer "F.SilkS")
+			(hide yes)
 			(effects
 				(font
@@
 			(at 0 3.2 0)
 			(layer "F.Fab")
+			(hide yes)
 			(effects
 				(font
@@
 			(at 0 -3.2 0)
 			(layer "F.SilkS")
+			(hide yes)
 			(effects
 				(font
@@
 			(at 0 3.2 0)
 			(layer "F.Fab")
+			(hide yes)
 			(effects
 				(font
@@
 		(net 18)
 	)
-	(segment
-		(start 138.46 64.0575)
-		(end 138.46 64.906875)
-		(width 0.2)
-		(layer "B.Cu")
-		(net 18)
-	)
-	(segment
-		(start 139.34125 63.17625)
-		(end 138.46 64.0575)
-		(width 0.2)
-		(layer "B.Cu")
-		(net 18)
-	)

Commit message: sch and pcb updates
Connections:
- U1 pad 10: unconnected-(U1-9-Pad10) -> Net-(J1-SDA)
- U1 pad 12: Net-(J1-SCL) -> unconnected-(U1-11-Pad12)
- U1 pad 13: Net-(J1-SDA) -> unconnected-(U1-12-Pad13)
- U1 pad 9: unconnected-(U1-8-Pad9) -> Net-(J1-SCL)
Routing:
- net Net-(J1-SCL): track 16.3 -> 24.0 mm
- net Net-(J1-SDA): track 12.8 -> 20.4 mm
Changed lines of the file:
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@@
 	(net 28 "Net-(U1-26)")
 	(net 29 "Net-(U1-27)")
-	(net 30 "unconnected-(U1-8-Pad9)")
+	(net 30 "unconnected-(U1-12-Pad13)")
 	(net 31 "Net-(U1-14)")
 	(net 32 "Net-(U1-15)")
@@
 	(net 34 "unconnected-(U1-29-Pad20)")
 	(net 35 "unconnected-(U1-28-Pad19)")
-	(net 36 "unconnected-(U1-9-Pad10)")
+	(net 36 "unconnected-(U1-11-Pad12)")
 	(net 37 "unconnected-(U1-10-Pad11)")
 	(footprint "ScottoKeebs_Hotswap:Hotswap_MX_1.00u"
@@
 			(layers "*.Cu" "*.Mask")
 			(remove_unused_layers no)
-			(net 30 "unconnected-(U1-8-Pad9)")
+			(net 20 "Net-(J1-SCL)")
 			(pinfunction "8")
 			(pintype "bidirectional")
@@
 			(layers "*.Cu" "*.Mask")
 			(remove_unused_layers no)
-			(net 36 "unconnected-(U1-9-Pad10)")
+			(net 22 "Net-(J1-SDA)")
 			(pinfunction "9")
 			(pintype "bidirectional")
@@
 			(layers "*.Cu" "*.Mask")
 			(remove_unused_layers no)
-			(net 20 "Net-(J1-SCL)")
+			(net 36 "unconnected-(U1-11-Pad12)")
 			(pinfunction "11")
 			(pintype "bidirectional")
@@
 			(layers "*.Cu" "*.Mask")
 			(remove_unused_layers no)
-			(net 22 "Net-(J1-SDA)")
+			(net 30 "unconnected-(U1-12-Pad13)")
 			(pinfunction "12")
 			(pintype "bidirectional")
@@
 	)
 	(segment
-		(start 153.53125 49.42625)
-		(end 159.66125 55.55625)
+		(start 153.53125 42.735)
+		(end 153.53125 57.04625)
 		(width 0.2)
 		(layer "F.Cu")
@@
 	)
 	(segment
-		(start 153.53125 42.735)
-		(end 153.53125 49.42625)
+		(start 153.53125 57.04625)
+		(end 159.66125 63.17625)
 		(width 0.2)
 		(layer "F.Cu")
@@
 	)
 	(segment
-		(start 155.63125 48.98625)
-		(end 159.66125 53.01625)
+		(start 155.375 42.03875)
+		(end 156.07125 42.735)
 		(width 0.2)
 		(layer "F.Cu")
@@
 	)
 	(segment
-		(start 155.63125 42.295)
-		(end 155.63125 48.98625)
+		(start 156.07125 42.735)
+		(end 156.07125 57.04625)
 		(width 0.2)
 		(layer "F.Cu")
@@
 	)
 	(segment
-		(start 155.375 42.03875)
-		(end 155.63125 42.295)
+		(start 156.07125 57.04625)
+		(end 159.66125 60.63625)
 		(width 0.2)
 		(layer "F.Cu")
