File: Boopsie v1 Kicad Files/Boopsie v1.kicad_sch (KiCad schematic)
At the start: 34 parts, among them J1 OLED_128x64, SW1 RotaryEncoder_Switch, SW2 RotaryEncoder_Switch, U1 RP2040_Zero

Commit message: sch and pcb updates
Connections:
- net at U1.10 (9): now also J1.4 (SDA)
- net at U1.12 (11): no longer J1.3 (SCL)
- net at U1.13 (12): no longer J1.4 (SDA)
- net at U1.9 (8): now also J1.3 (SCL)
Other:
- moved on the sheet: J1
Changed lines of the file:
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@@
-	(wire
-		(pts
-			(xy 139.7 85.09) (xy 114.3 85.09)
-		)
-		(stroke
-			(width 0)
-			(type default)
-		)
-	)
 	(wire
 		(pts
@@
 	(wire
 		(pts
-			(xy 139.7 85.09) (xy 139.7 72.39)
-		)
-		(stroke
-			(width 0)
-			(type default)
-		)
-	)
-	(wire
-		(pts
 			(xy 125.73 111.76) (xy 125.73 120.65)
 		)
@@
 	(wire
 		(pts
-			(xy 114.3 82.55) (xy 113.03 82.55)
-		)
-		(stroke
-			(width 0)
-			(type default)
-		)
-	)
-	(wire
-		(pts
 			(xy 92.71 97.79) (xy 92.71 133.35)
 		)
@@
 	(wire
 		(pts
-			(xy 114.3 85.09) (xy 114.3 82.55)
-		)
-		(stroke
-			(width 0)
-			(type default)
-		)
-	)
-	(wire
-		(pts
 			(xy 161.29 68.58) (xy 161.29 72.39)
 		)
@@
 	(wire
 		(pts
-			(xy 128.27 62.23) (xy 128.27 72.39)
-		)
-		(stroke
-			(width 0)
-			(type default)
-		)
-	)
-	(wire
-		(pts
-			(xy 113.03 86.36) (xy 140.97 86.36)
-		)
-		(stroke
-			(width 0)
-			(type default)
-		)
-	)
-	(wire
-		(pts
-			(xy 140.97 86.36) (xy 140.97 71.12)
+			(xy 130.81 62.23) (xy 130.81 76.2)
 		)
 		(stroke
@@
 	(wire
 		(pts
-			(xy 130.81 71.12) (xy 130.81 72.39)
-		)
-		(stroke
-			(width 0)
-			(type default)
-		)
-	)
-	(wire
-		(pts
 			(xy 195.58 71.12) (xy 195.58 72.39)
 		)
@@
 	(wire
 		(pts
-			(xy 92.71 62.23) (xy 128.27 62.23)
+			(xy 92.71 62.23) (xy 130.81 62.23)
+		)
+		(stroke
+			(width 0)
+			(type default)
+		)
+	)
+	(wire
+		(pts
+			(xy 135.89 90.17) (xy 135.89 76.2)
 		)
 		(stroke
@@
 	(wire
 		(pts
-			(xy 125.73 71.12) (xy 125.73 72.39)
+			(xy 128.27 71.12) (xy 128.27 76.2)
 		)
 		(stroke
@@
 	(wire
 		(pts
+			(xy 113.03 90.17) (xy 135.89 90.17)
+		)
+		(stroke
+			(width 0)
+			(type default)
+		)
+	)
+	(wire
+		(pts
 			(xy 125.73 139.7) (xy 125.73 158.75)
 		)
@@
 	(wire
 		(pts
-			(xy 140.97 71.12) (xy 130.81 71.12)
-		)
-		(stroke
-			(width 0)
-			(type default)
-		)
-	)
-	(wire
-		(pts
 			(xy 92.71 133.35) (xy 100.33 133.35)
 		)
@@
 	(wire
 		(pts
-			(xy 139.7 72.39) (xy 133.35 72.39)
-		)
-		(stroke
-			(width 0)
-			(type default)
-		)
-	)
-	(wire
-		(pts
 			(xy 193.04 66.04) (xy 193.04 72.39)
 		)
@@
 	(wire
 		(pts
+			(xy 128.27 71.12) (xy 125.73 71.12)
+		)
+		(stroke
+			(width 0)
+			(type default)
+		)
+	)
+	(wire
+		(pts
 			(xy 115.57 113.03) (xy 115.57 120.65)
 		)
@@
 	(wire
 		(pts
+			(xy 107.95 97.79) (xy 133.35 97.79)
+		)
+		(stroke
+			(width 0)
+			(type default)
+		)
+	)
+	(wire
+		(pts
 			(xy 161.29 111.76) (xy 161.29 113.03)
 		)
@@
 	(wire
 		(pts
-			(xy 113.03 86.36) (xy 113.03 85.09)
-		)
-		(stroke
-			(width 0)
-			(type default)
-		)
-	)
-	(wire
-		(pts
 			(xy 100.33 152.4) (xy 110.49 152.4)
 		)
@@
 		(pts
 			(xy 193.04 95.25) (xy 193.04 102.87)
+		)
+		(stroke
+			(width 0)
+			(type default)
+		)
+	)
+	(wire
+		(pts
+			(xy 133.35 97.79) (xy 133.35 76.2)
 		)
 		(stroke
@@
 	(symbol
 		(lib_id "ScottoKeebs:OLED_128x64")
-		(at 129.54 74.93 0)
+		(at 132.08 78.74 0)
 		(unit 1)
 		(exclude_from_sim no)
@@
 		(fields_autoplaced yes)
 		(property "Reference" "J1"
-			(at 140.97 78.7399 0)
+			(at 143.51 82.5499 0)
 			(effects
 				(font
@@
 		)
 		(property "Value" "OLED_128x64"
-			(at 140.97 81.2799 0)
+			(at 143.51 85.0899 0)
 			(effects
 				(font
@@
 		)
 		(property "Footprint" "ScottoKeebs_Components:OLED_128x64"
-			(at 129.54 88.9 0)
+			(at 132.08 92.71 0)
 			(effects
 				(font
@@
 		)
 		(property "Datasheet" ""
-			(at 130.81 74.93 90)
+			(at 133.35 78.74 90)
 			(effects
 				(font
@@
 		)
 		(property "Description" ""
-			(at 129.54 74.93 0)
-			(effects
-				(font
+			(at 132.08 78.74 0)
+			(effects
+				(font

Commit message: final final
Connections:
- net at S12.1, S4.1, S8.1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: no longer SW1.S1
- net at S11.1, S3.1, S7.1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: now also SW1.S1
Changed lines of the file:
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@@
+	)
+	(junction
+		(at 115.57 114.3)
+		(diameter 0)
+		(color 0 0 0 0)
 	)
 	(junction
@@
 	)
 	(junction
-		(at 161.29 111.76)
-		(diameter 0)
-		(color 0 0 0 0)
-	)
-	(junction
 		(at 158.75 71.12)
 		(diameter 0)
@@
 	(wire
 		(pts
+			(xy 115.57 114.3) (xy 198.12 114.3)
+		)
+		(stroke
+			(width 0)
+			(type default)
+		)
+	)
+	(wire
+		(pts
 			(xy 105.41 72.39) (xy 105.41 68.58)
 		)
@@
 	(wire
 		(pts
+			(xy 115.57 114.3) (xy 115.57 120.65)
+		)
+		(stroke
+			(width 0)
+			(type default)
+		)
+	)
+	(wire
+		(pts
 			(xy 156.21 104.14) (xy 156.21 102.87)
 		)
@@
 	(wire
 		(pts
-			(xy 115.57 113.03) (xy 115.57 120.65)
+			(xy 115.57 113.03) (xy 115.57 114.3)
 		)
 		(stroke
@@
 	(wire
 		(pts
-			(xy 161.29 111.76) (xy 161.29 113.03)
-		)
-		(stroke
-			(width 0)
-			(type default)
-		)
-	)
-	(wire
-		(pts
 			(xy 156.21 102.87) (xy 193.04 102.87)
 		)
@@
 	(wire
 		(pts
+			(xy 198.12 87.63) (xy 198.12 114.3)
+		)
+		(stroke
+			(width 0)
+			(type default)
+		)
+	)
+	(wire
+		(pts
+			(xy 193.04 95.25) (xy 193.04 102.87)
+		)
+		(stroke
+			(width 0)
+			(type default)
+		)
+	)
+	(wire
+		(pts
+			(xy 133.35 97.79) (xy 133.35 76.2)
+		)
+		(stroke
+			(width 0)
+			(type default)
+		)
+	)
+	(wire
+		(pts
 			(xy 161.29 87.63) (xy 161.29 111.76)
 		)
 		(stroke
-			(width 0)
-			(type default)
-		)
-	)
-	(wire
-		(pts
-			(xy 198.12 113.03) (xy 198.12 87.63)
-		)
-		(stroke
-			(width 0)
-			(type default)
-		)
-	)
-	(wire
-		(pts
-			(xy 193.04 95.25) (xy 193.04 102.87)
-		)
-		(stroke
-			(width 0)
-			(type default)
-		)
-	)
-	(wire
-		(pts
-			(xy 133.35 97.79) (xy 133.35 76.2)
-		)
-		(stroke
-			(width 0)
-			(type default)
-		)
-	)
-	(wire
-		(pts
-			(xy 161.29 113.03) (xy 198.12 113.03)
-		)
-		(stroke
